Commit message: Added Gazebo setup

File: tiago_autonomy_bringup/urdf/tiago_autonomy.urdf (robot description, URDF)
Before this commit: robot tiago_dual, 85 links, 84 joints
Links:
- link arm_left_tool_link: mass 0.1 -> 0.01
- link arm_right_tool_link: mass 0.1 -> 0.01
Joints:
- joint caster_back_left_1_joint: origin xyz=-0.17350000000000002 0.102 -0.0335 rpy=0 0 0 -> xyz=-0.1735 0.102 -0.0335 rpy=0 0 0
- joint caster_back_right_1_joint: origin xyz=-0.17350000000000002 -0.102 -0.0335 rpy=0 0 0 -> xyz=-0.1735 -0.102 -0.0335 rpy=0 0 0
- joint torso_fixed_column_joint: axis 0 0 0 -> (none)
- joint torso_fixed_joint: axis 0 0 0 -> (none)

Commit message: Add EKF configuration and navigation launch files for TIAGo
- Updated CMakeLists.txt to include maps directory in installation.
- Modified ekf.yaml to use quoted frame names for consistency.
- Enhanced tiago_navigation.launch.py to include navigation parameters and map file.
- Added apartment_map.pgm and apartment_map.yaml for the navigation setup.

File: tiago_autonomy_bringup/urdf/tiago_autonomy.urdf (robot description, URDF)
Before this commit: robot tiago_dual, 85 links, 84 joints
Links:
- removed link head_front_camera_optical_frame
- link gripper_left_left_inner_finger: mass 0.0104003125914103 -> 0.01040
- link gripper_left_left_inner_knuckle: mass 0.0271177346495152 -> 0.02711
- link gripper_left_left_outer_finger: mass 0.022614240507152 -> 0.02261
- link gripper_left_left_outer_knuckle: mass 0.00853198276973456 -> 0.00853
- link gripper_left_right_inner_finger: mass 0.0104003125914103 -> 0.01040
- link gripper_left_right_inner_knuckle: mass 0.0271177346495152 -> 0.02711
- link gripper_left_right_outer_finger: mass 0.022614240507152 -> 0.02261
- link gripper_left_right_outer_knuckle: mass 0.00853198276973456 -> 0.00853
- link gripper_right_left_inner_finger: mass 0.0104003125914103 -> 0.01040
- link gripper_right_left_inner_knuckle: mass 0.0271177346495152 -> 0.02711
- link gripper_right_left_outer_finger: mass 0.022614240507152 -> 0.02261
- link gripper_right_left_outer_knuckle: mass 0.00853198276973456 -> 0.00853
- link gripper_right_right_inner_finger: mass 0.0104003125914103 -> 0.01040
- link gripper_right_right_inner_knuckle: mass 0.0271177346495152 -> 0.02711
- link gripper_right_right_outer_finger: mass 0.022614240507152 -> 0.02261
- link gripper_right_right_outer_knuckle: mass 0.00853198276973456 -> 0.00853
- link head_front_camera_link: mass 0.21970000000 -> 0.2197
- link suspension_left_link: mass 10 -> 0.5
- link suspension_right_link: mass 10 -> 0.5
Joints:
- removed joint head_front_camera_optical_joint
- joint torso_lift_joint: origin xyz=0.0 0.0 0.597 rpy=0.0 0.0 0.0 -> xyz=0.0 0.0 0.597 rpy=0 0 0
- joint wheel_left_joint: limit effort=6.0 velocity=100.0 -> effort=50.0 velocity=10.0
- joint wheel_right_joint: limit effort=6.0 velocity=100.0 -> effort=50.0 velocity=10.0
