Commit message: Add URDF to occupancy grid conversion script and update navigation configurations
- Introduced a new script `urdf_to_map.py` for generating occupancy grids from URDF collision geometries.
- Updated `CMakeLists.txt` to install the new `dock_pose_publisher.py` script.
- Added `apriltag_dock.yaml` configuration for AprilTag detection parameters.
- Modified `ekf.yaml` to reduce the EKF frequency from 30.0 to 20.0.
- Created `nav2_tiago_params.yaml` with comprehensive navigation parameters for AMCL, planners, and controllers.
- Updated launch file to include AprilTag detection and dock pose publishing nodes.
- Adjusted `apartment_map.yaml` to correct the origin and maintain consistency with the generated map.
- Added `dock_pose_publisher.py` to publish detected dock poses based on AprilTag transformations.
- Removed the unused `tiago_navigation.cpp` source file.

File: tiago_autonomy_bringup/urdf/apartment.urdf (robot description, URDF)
Before this commit: robot apartment, 118 links, 117 joints
Links:
- added link dock_apriltag_link; visual box size=0.002 0.18 0.18
- added link docking_station_link; collision box size=0.12 0.40 0.25; visual box size=0.12 0.40 0.25
Joints:
- added joint dock_apriltag_joint: type fixed, parent apartment_root, child dock_apriltag_link, origin xyz=8.17 4.93 0.70 rpy=0 0 1.5708
- added joint docking_station_joint: type fixed, parent apartment_root, child docking_station_link, origin xyz=8.17 4.85 0.0 rpy=0 0 1.5708

Commit message: Refactor TIAGo Navigation Launch and Add Real-Time Controllers
- Updated `tiago_navigation.launch.py` to improve organization and readability.
- Added new nodes for docking server, static TF publisher, and velocity relay.
- Adjusted parameters to use LaunchConfiguration for better flexibility.
- Modified `apartment_map.yaml` to correct the origin coordinates.
- Enhanced `dock_pose_publisher.py` to include dynamic parameters and improved pose publishing logic.
- Introduced `twist_to_twiststamped.py` for relaying Twist messages as TwistStamped.
- Created `tiago_rtt_controllers` package with real-time Cartesian controllers for TIAGo.
- Implemented `tiago_cartesian_controller.cpp` for managing arm joint states and Cartesian control.
- Added launch file `tiago_realtime_control.launch.py` to manage controller lifecycle and deployment.
- Configured CMake and package.xml for the new RTT controllers package.

File: tiago_autonomy_bringup/urdf/apartment.urdf (robot description, URDF)
Before this commit: robot apartment, 120 links, 119 joints
Joints:
- joint dock_apriltag_joint: origin xyz=8.17 4.93 0.70 rpy=0 0 1.5708 -> xyz=0.14 0.0 0.70 rpy=0 0 0; parent apartment_root -> docking_station_link
- joint docking_station_joint: origin xyz=8.17 4.85 0.0 rpy=0 0 1.5708 -> xyz=8.17 4.79 0.0 rpy=0 0 1.5708
